Commit message: Changed id's to strings and added leg inverse kinematics

File: robot/urdf/ardent.urdf (robot description, URDF)
Before this commit: robot ardent, 26 links, 25 joints
Links:
- removed link c1_lf
- removed link c1_lm
- removed link c1_lr
- removed link c1_rf
- removed link c1_rm
- removed link c1_rr
- added link coxa_lf, mass 0.024357719; collision box size=0.022 0.045 0.0325; visual box size=0.022 0.045 0.0325
- added link coxa_lm, mass 0.024357719; collision box size=0.022 0.045 0.0325; visual box size=0.022 0.045 0.0325
- added link coxa_lr, mass 0.024357719; collision box size=0.022 0.045 0.0325; visual box size=0.022 0.045 0.0325
- added link coxa_rf, mass 0.024357719; collision box size=0.022 0.045 0.0325; visual box size=0.022 0.045 0.0325
- added link coxa_rm, mass 0.024357719; collision box size=0.022 0.045 0.0325; visual box size=0.022 0.045 0.0325
- added link coxa_rr, mass 0.024357719; collision box size=0.022 0.045 0.0325; visual box size=0.022 0.045 0.0325
Joints:
- removed joint j_c1_lf
- removed joint j_c1_lm
- removed joint j_c1_lr
- removed joint j_c1_rf
- removed joint j_c1_rm
- removed joint j_c1_rr
- added joint j_coxa_lf: type revolute, parent MP_BODY, child coxa_lf, origin xyz=0.175 0.1  0.001116 rpy=0 0 0.765, axis 0 0 1, limit lower=-3.14 upper=3.14 effort=20 velocity=2
- added joint j_coxa_lm: type revolute, parent MP_BODY, child coxa_lm, origin xyz=0 0.2  0.001116 rpy=0 0 1.57, axis 0 0 1, limit lower=-3.14 upper=3.14 effort=20 velocity=2
- added joint j_coxa_lr: type revolute, parent MP_BODY, child coxa_lr, origin xyz=-0.175 0.1  0.001116 rpy=0 0 2.335, axis 0 0 1, limit lower=-3.14 upper=3.14 effort=20 velocity=2
- added joint j_coxa_rf: type revolute, parent MP_BODY, child coxa_rf, origin xyz=0.175 -0.1  0.001116 rpy=0 0 5.475, axis 0 0 1, limit lower=-3.14 upper=3.14 effort=20 velocity=2
- added joint j_coxa_rm: type revolute, parent MP_BODY, child coxa_rm, origin xyz=0 -0.2  0.001116 rpy=0 0 -1.57, axis 0 0 1, limit lower=-3.14 upper=3.14 effort=20 velocity=2
- added joint j_coxa_rr: type revolute, parent MP_BODY, child coxa_rr, origin xyz=-0.175 -0.1  0.001116 rpy=0 0 -2.335, axis 0 0 1, limit lower=-3.14 upper=3.14 effort=20 velocity=2
- joint j_c2_lf: parent c1_lf -> coxa_lf
- joint j_c2_lm: parent c1_lm -> coxa_lm
- joint j_c2_lr: parent c1_lr -> coxa_lr
- joint j_c2_rf: parent c1_rf -> coxa_rf
- joint j_c2_rm: parent c1_rm -> coxa_rm
- joint j_c2_rr: parent c1_rr -> coxa_rr

File: robot/urdf/ardent_urdf.xacro (robot description, xacro)
@@ -49,5 +49,5 @@
 </xacro:macro>
  <xacro:macro name="leg_l" params="xyz rpy suffix">
-  <link name="c1_${suffix}">
+  <link name="coxa_${suffix}">
     <inertial>
       <origin xyz="0 0 0" rpy="0 0 0"  />
@@ -149,7 +149,7 @@
     </collision>
   </link>
-<joint name="j_c1_${suffix}" type="revolute">
+<joint name="j_coxa_${suffix}" type="revolute">
     <parent link="MP_BODY"/>
-    <child link="c1_${suffix}"/>
+    <child link="coxa_${suffix}"/>
     <origin xyz="${xyz}" rpy="${rpy}" />
     <axis xyz="0 0 1" />
@@ -157,5 +157,5 @@
   </joint>
   <joint name="j_c2_${suffix}" type="fixed">
-    <parent link="c1_${suffix}"/>
+    <parent link="coxa_${suffix}"/>
     <child link="c2_${suffix}"/>
     <origin xyz="0.0135 0 0" rpy="0 0 0" />
@@ -203,7 +203,7 @@
     </collision>
     </gazebo> -->
-  <!-- <joint name="j_c1_${suffix}" type="revolute">
+  <!-- <joint name="j_coxa_${suffix}" type="revolute">
     <parent link="MP_BODY"/>
-    <child link="c1_${suffix}"/>
+    <child link="coxa_${suffix}"/>
     <origin xyz="${xyz}" rpy="${rpy}" />
     <axis xyz="1 0 0" />
@@ -211,5 +211,5 @@
   </joint>
   <joint name="j_c2_${suffix}" type="fixed">
-    <parent link="c1_${suffix}"/>
+    <parent link="coxa_${suffix}"/>
     <child link="c2_${suffix}"/>
     <origin xyz="0 -0.033 0" rpy="0 1.5704 3.14159" />
@@ -229,10 +229,10 @@
     <limit effort="2.8" velocity="5.6548668" lower="-2.6179939" upper="2.6179939" />
   </joint> -->
-   <transmission name="t_c1_${suffix}">
+   <transmission name="t_coxa_${suffix}">
     <type>transmission_interface/SimpleTransmission</type>
-    <joint name="j_c1_${suffix}">
-      <hardwareInterface>hardware_interface/EffortJointInterface</hardwareInterface>
-    </joint>
-    <actuator name="m_c1_${suffix}">
+    <joint name="j_coxa_${suffix}">
+      <hardwareInterface>hardware_interface/EffortJointInterface</hardwareInterface>
+    </joint>
+    <actuator name="m_coxa_${suffix}">
       <hardwareInterface>hardware_interface/EffortJointInterface</hardwareInterface>
       <mechanicalReduction>1</mechanicalReduction>
@@ -262,5 +262,5 @@
     <material>Gazebo/Orange</material>
   </gazebo>
-  <gazebo reference="c1_${suffix}">
+  <gazebo reference="coxa_${suffix}">
     <material>Gazebo/Black</material>
   </gazebo>

Commit message: removed namespace (temporary) and adding visualization

File: robot/urdf/ardent.urdf (robot description, URDF)
Before this commit: robot ardent, 26 links, 25 joints
Joints:
- joint j_c2_lf: limit (none) -> lower=-3.14 upper=3.14 effort=30 velocity=0.5
- joint j_c2_lm: limit (none) -> lower=-3.14 upper=3.14 effort=30 velocity=0.5
- joint j_c2_lr: limit (none) -> lower=-3.14 upper=3.14 effort=30 velocity=0.5
- joint j_c2_rf: limit (none) -> lower=-3.14 upper=3.14 effort=30 velocity=0.5
- joint j_c2_rm: limit (none) -> lower=-3.14 upper=3.14 effort=30 velocity=0.5
- joint j_c2_rr: limit (none) -> lower=-3.14 upper=3.14 effort=30 velocity=0.5
- joint j_coxa_lf: limit lower=-3.14 upper=3.14 effort=20 velocity=2 -> lower=-3.14 upper=3.14 effort=30 velocity=0.5
- joint j_coxa_lm: limit lower=-3.14 upper=3.14 effort=20 velocity=2 -> lower=-3.14 upper=3.14 effort=30 velocity=0.5
- joint j_coxa_lr: limit lower=-3.14 upper=3.14 effort=20 velocity=2 -> lower=-3.14 upper=3.14 effort=30 velocity=0.5
- joint j_coxa_rf: limit lower=-3.14 upper=3.14 effort=20 velocity=2 -> lower=-3.14 upper=3.14 effort=30 velocity=0.5
- joint j_coxa_rm: limit lower=-3.14 upper=3.14 effort=20 velocity=2 -> lower=-3.14 upper=3.14 effort=30 velocity=0.5
- joint j_coxa_rr: limit lower=-3.14 upper=3.14 effort=20 velocity=2 -> lower=-3.14 upper=3.14 effort=30 velocity=0.5
- joint j_femur_lf: limit lower=-3.14 upper=3.14 effort=20 velocity=2 -> lower=-3.14 upper=3.14 effort=30 velocity=0.5
- joint j_femur_lm: limit lower=-3.14 upper=3.14 effort=20 velocity=2 -> lower=-3.14 upper=3.14 effort=30 velocity=0.5
- joint j_femur_lr: limit lower=-3.14 upper=3.14 effort=20 velocity=2 -> lower=-3.14 upper=3.14 effort=30 velocity=0.5
- joint j_femur_rf: limit lower=-3.14 upper=3.14 effort=20 velocity=2 -> lower=-3.14 upper=3.14 effort=30 velocity=0.5
- joint j_femur_rm: limit lower=-3.14 upper=3.14 effort=20 velocity=2 -> lower=-3.14 upper=3.14 effort=30 velocity=0.5
- joint j_femur_rr: limit lower=-3.14 upper=3.14 effort=20 velocity=2 -> lower=-3.14 upper=3.14 effort=30 velocity=0.5
- joint j_tibia_lf: limit lower=-2.6179939 upper=2.6179939 effort=20 velocity=2 -> lower=-3.14 upper=3.14 effort=30 velocity=0.5
- joint j_tibia_lm: limit lower=-2.6179939 upper=2.6179939 effort=20 velocity=2 -> lower=-3.14 upper=3.14 effort=30 velocity=0.5
- joint j_tibia_lr: limit lower=-2.6179939 upper=2.6179939 effort=20 velocity=2 -> lower=-3.14 upper=3.14 effort=30 velocity=0.5
- joint j_tibia_rf: limit lower=-2.6179939 upper=2.6179939 effort=20 velocity=2 -> lower=-3.14 upper=3.14 effort=30 velocity=0.5
- joint j_tibia_rm: limit lower=-2.6179939 upper=2.6179939 effort=20 velocity=2 -> lower=-3.14 upper=3.14 effort=30 velocity=0.5
- joint j_tibia_rr: limit lower=-2.6179939 upper=2.6179939 effort=20 velocity=2 -> lower=-3.14 upper=3.14 effort=30 velocity=0.5

File: robot/urdf/ardent.xacro (robot description, xacro)
@@ -8,5 +8,5 @@
    <gazebo>
     <plugin filename="libgazebo_ros_control.so" name="gazebo_ros_control">
-      <robotNamespace>/ardent</robotNamespace>
+      <!-- <robotNamespace>/ardent</robotNamespace> -->
     </plugin>
   </gazebo>

File: robot/urdf/ardent_urdf.xacro (robot description, xacro)
@@ -101,5 +101,6 @@
       <origin xyz="1 0 0" rpy="0 0 0"  />
       <mass value="0.0286"/>
-     <inertia ixx="0.000035572"  ixy="-0.000114256"  ixz="-0.000008584" iyy="0.000756486" iyz="-0.000001714" izz="0.000791714" />
+     <!-- <inertia ixx="0.000035572"  ixy="-0.000114256"  ixz="-0.000008584" iyy="0.000756486" iyz="-0.000001714" izz="0.000791714" /> -->
+     <inertia ixx="0.00059"  ixy="-0.0"  ixz="-0.0" iyy="0.0" iyz="-0.0" izz="0.00059" />
     </inertial>
     <visual>
@@ -128,5 +129,6 @@
       <!-- g/mm^2 -->
      <!-- <inertia ixx="35572"  ixy="-114256"  ixz="-8584" iyy="756486" iyz="-1714" izz="791714" /> -->
-     <inertia ixx="0.000035572"  ixy="-0.000114256"  ixz="-0.000008584" iyy="0.000756486" iyz="-0.000001714" izz="0.000791714" />
+     <!-- <inertia ixx="0.000035572"  ixy="-0.000114256"  ixz="-0.000008584" iyy="0.000756486" iyz="-0.000001714" izz="0.000791714" /> -->
+     <inertia ixx="0.00059"  ixy="-0.0"  ixz="-0.0" iyy="0.0" iyz="-0.0" izz="0.00059" />
     </inertial>
     <visual>
@@ -154,5 +156,5 @@
     <origin xyz="${xyz}" rpy="${rpy}" />
     <axis xyz="0 0 1" />
-    <limit effort="20" velocity="2" lower="-3.14" upper="3.14" />
+    <limit effort="30" velocity="0.5" lower="-3.14" upper="3.14" />
   </joint>
   <joint name="j_c2_${suffix}" type="fixed">
@@ -160,4 +162,5 @@
     <child link="c2_${suffix}"/>
     <origin xyz="0.0135 0 0" rpy="0 0 0" />
+    <limit effort="30" velocity="0.5" lower="-3.14" upper="3.14" />
   </joint>
   <joint name="j_femur_${suffix}" type="revolute">
@@ -166,5 +169,5 @@
     <origin xyz="0 0 0" rpy=" 1.57 0 0" />
     <axis xyz="0 0 1" />
-    <limit effort="20" velocity="2" lower="-3.14" upper="3.14" />
+    <limit effort="30" velocity="0.5" lower="-3.14" upper="3.14" />
   </joint>
   <joint name="j_tibia_${suffix}" type="revolute">
@@ -173,5 +176,5 @@
     <origin xyz="0.25 0 0" rpy="0 0 0" />
     <axis xyz="0 0 1" />
-    <limit effort="20" velocity="2" lower="-2.6179939" upper="2.6179939" />
+    <limit effort="30" velocity="0.5" lower="-3.14" upper="3.14" />
   </joint>
    <!-- <gazebo reference="$tibia_${suffix}">

Commit message: Updated robot model for new masses and dimensions

File: robot/urdf/ardent.urdf (robot description, URDF)
Before this commit: robot ardent, 26 links, 25 joints
Links:
- link femur_lf: geometry collision cylinder length=0.15 radius=0.015; visual cylinder length=0.15 radius=0.015
- link femur_lm: geometry collision cylinder length=0.15 radius=0.015; visual cylinder length=0.15 radius=0.015
- link femur_lr: geometry collision cylinder length=0.15 radius=0.015; visual cylinder length=0.15 radius=0.015
- link femur_rf: geometry collision cylinder length=0.15 radius=0.015; visual cylinder length=0.15 radius=0.015
- link femur_rm: geometry collision cylinder length=0.15 radius=0.015; visual cylinder length=0.15 radius=0.015
- link femur_rr: geometry collision cylinder length=0.15 radius=0.015; visual cylinder length=0.15 radius=0.015
Joints:
- joint j_coxa_lf: origin xyz=0.175 0.1  0.001116 rpy=0 0 0.765 -> xyz=0.175 0.1  0.001116 rpy=0 0 0.52
- joint j_coxa_lr: origin xyz=-0.175 0.1  0.001116 rpy=0 0 2.335 -> xyz=-0.175 0.1  0.001116 rpy=0 0 2.62
- joint j_coxa_rf: origin xyz=0.175 -0.1  0.001116 rpy=0 0 5.475 -> xyz=0.175 -0.1  0.001116 rpy=0 0 5.576
- joint j_coxa_rr: origin xyz=-0.175 -0.1  0.001116 rpy=0 0 -2.335 -> xyz=-0.175 -0.1  0.001116 rpy=0 0 -2.62
- joint j_tibia_lf: origin xyz=0.25 0 0 rpy=0 0 0 -> xyz=0.125 0 0 rpy=0 0 0
- joint j_tibia_lm: origin xyz=0.25 0 0 rpy=0 0 0 -> xyz=0.125 0 0 rpy=0 0 0
- joint j_tibia_lr: origin xyz=0.25 0 0 rpy=0 0 0 -> xyz=0.125 0 0 rpy=0 0 0
- joint j_tibia_rf: origin xyz=0.25 0 0 rpy=0 0 0 -> xyz=0.125 0 0 rpy=0 0 0
- joint j_tibia_rm: origin xyz=0.25 0 0 rpy=0 0 0 -> xyz=0.125 0 0 rpy=0 0 0
- joint j_tibia_rr: origin xyz=0.25 0 0 rpy=0 0 0 -> xyz=0.125 0 0 rpy=0 0 0

File: robot/urdf/ardent_urdf.xacro (robot description, xacro)
@@ -51,10 +51,10 @@
       </transmission> -->
     <!-- Build Leg -->
-    <xacro:leg_l xyz="0.175 -0.1  0.001116"  rpy="0 0 5.475" suffix="rf"/>
+    <xacro:leg_l xyz="0.175 -0.1  0.001116"  rpy="0 0 5.576" suffix="rf"/>
     <xacro:leg_l xyz="0 -0.2  0.001116"  rpy="0 0 -1.57" suffix="rm"/>
-    <xacro:leg_l xyz="-0.175 -0.1  0.001116"  rpy="0 0 -2.335" suffix="rr"/>
-    <xacro:leg_l xyz="0.175 0.1  0.001116"  rpy="0 0 0.765" suffix="lf"/>
+    <xacro:leg_l xyz="-0.175 -0.1  0.001116"  rpy="0 0 -2.62" suffix="rr"/>
+    <xacro:leg_l xyz="0.175 0.1  0.001116"  rpy="0 0 0.52" suffix="lf"/>
     <xacro:leg_l xyz="0 0.2  0.001116"  rpy="0 0 1.57" suffix="lm"/>
-    <xacro:leg_l xyz="-0.175 0.1  0.001116"  rpy="0 0 2.335" suffix="lr"/>
+    <xacro:leg_l xyz="-0.175 0.1  0.001116"  rpy="0 0 2.62" suffix="lr"/>
 </xacro:macro>
  <xacro:macro name="leg_l" params="xyz rpy suffix">
@@ -115,8 +115,8 @@
     </inertial>
     <visual>
-      <origin xyz="0.125 0 0" rpy="0 1.57 0"  />
+      <origin xyz="0.075 0 0" rpy="0 1.57 0"  />
       <geometry>
         <!-- <box size="0.022 0.25 0.0325" /> -->
-        <cylinder  radius="0.015" length="0.25" />
+        <cylinder  radius="0.015" length="0.15" />
         <!--<mesh filename="package://phantomx_description/meshes/thigh_l.STL"  scale="1 1 1"/>-->
       </geometry>
@@ -126,7 +126,7 @@
     </visual>
     <collision>
-      <origin xyz="0.125 0 0" rpy="0 1.57 0"  />
-      <geometry>
-        <cylinder  radius="0.015" length="0.25" />
+      <origin xyz="0.075 0 0" rpy="0 1.57 0"  />
+      <geometry>
+        <cylinder  radius="0.015" length="0.15" />
         <!-- <mesh filename="package://phantomx_description/meshes/thigh_l_coll.STL"  scale="1 1 1"/> -->
       </geometry>
@@ -143,5 +143,5 @@
     </inertial>
     <visual>
-      <origin xyz="0.117 0 0" rpy="1.57 0 1.57"  />
+      <origin xyz="0.125 0 0" rpy="1.57 0 1.57"  />
       <geometry>
         <cylinder  radius="0.015" length="0.25" />
@@ -154,5 +154,5 @@
     </visual>
     <collision>
-      <origin xyz="0.117 0 0" rpy="1.57 0 1.57"  />
+      <origin xyz="0.125 0 0" rpy="1.57 0 1.57"  />
       <geometry>
         <cylinder  radius="0.015" length="0.25" />
@@ -184,5 +184,5 @@
     <parent link="femur_${suffix}"/>
     <child link="tibia_${suffix}"/>
-    <origin xyz="0.25 0 0" rpy="0 0 0" />
+    <origin xyz="0.125 0 0" rpy="0 0 0" />
     <axis xyz="0 0 1" />
     <limit effort="30" velocity="0.5" lower="-3.14" upper="3.14" />
