Commit message: Updated Inverse Kinematics

File: robot/urdf/ardent_urdf.xacro (robot description, xacro)
@@ -9,9 +9,4 @@
 <xacro:property name="joint_velocity" value ="100"/> -->
 <xacro:macro name="ardent" params="parent *origin">
-    <joint name="j_ardent_attachment" type="fixed">
-      <parent link="${parent}"/>
-      <child link="MP_BODY"/>
-      <xacro:insert_block name="origin" />
-    </joint>
     <link name="MP_BODY">
       <inertial>
@@ -40,4 +35,9 @@
       </collision>
     </link>
+    <joint name="j_ardent_attachment" type="fixed">
+      <parent link="${parent}"/>
+      <child link="MP_BODY"/>
+      <xacro:insert_block name="origin" />
+    </joint>
     <!-- Build Leg -->
     <xacro:leg_l xyz="0.175 -0.1  0.001116"  rpy="0 0 5.475" suffix="rf"/>

Commit message: fixed urdf to match IK

File: robot/urdf/ardent_urdf.xacro (robot description, xacro)
@@ -131,5 +131,5 @@
     </inertial>
     <visual>
-      <origin xyz="0 -0.117 0" rpy="1.57 0 0"  />
+      <origin xyz="0.117 0 0" rpy="1.57 0 1.57"  />
       <geometry>
         <cylinder  radius="0.015" length="0.25" />
@@ -142,5 +142,5 @@
     </visual>
     <collision>
-      <origin xyz="0 -0.117 0" rpy="1.57 0 0"  />
+      <origin xyz="0.117 0 0" rpy="1.57 0 1.57"  />
       <geometry>
         <cylinder  radius="0.015" length="0.25" />

Commit message: Edited controller to be based on trajectory instead of position

File: robot/urdf/ardent_urdf.xacro (robot description, xacro)
@@ -40,4 +40,14 @@
       <xacro:insert_block name="origin" />
     </joint>
+    <!-- <transmission name="t_ardent">
+        <type>transmission_interface/SimpleTransmission</type>
+        <joint name="j_ardent_attachment">
+          <hardwareInterface>hardware_interface/EffortJointInterface</hardwareInterface>
+        </joint>
+        <actuator name="j_ardent_attachment">
+          <hardwareInterface>hardware_interface/EffortJointInterface</hardwareInterface>
+          <mechanicalReduction>1</mechanicalReduction>
+        </actuator>
+      </transmission> -->
     <!-- Build Leg -->
     <xacro:leg_l xyz="0.175 -0.1  0.001116"  rpy="0 0 5.475" suffix="rf"/>

Commit message: Changed the gazebo urdf what will be ardent_model transmission

File: robot/urdf/ardent_urdf.xacro (robot description, xacro)
@@ -242,5 +242,23 @@
     <limit effort="2.8" velocity="5.6548668" lower="-2.6179939" upper="2.6179939" />
   </joint> -->
-   <transmission name="t_coxa_${suffix}">
+  <transmission type="ardent_model/SimpleTransmission" name="t_coxa_${suffix}">
+    <joint name="t_coxa_${suffix}">
+    <actuator name="t_coxa_${suffix}">
+    <mechanicalReduction>1</mechanicalReduction>
+    <!-- <compensator k_belt="4000.0" mass_motor="0.05" kd_motor="15.0" lambda_motor="40.0" lambda_joint="40.0" lambda_combined="0.0"/> -->
+  </transmission>
+  <transmission type="ardent_model/SimpleTransmission" name="t_femur_${suffix}">
+    <joint name="t_femur_${suffix}">
+    <actuator name="t_femur_${suffix}">
+    <mechanicalReduction>1</mechanicalReduction>
+    <!-- <compensator k_belt="4000.0" mass_motor="0.05" kd_motor="15.0" lambda_motor="40.0" lambda_joint="40.0" lambda_combined="0.0"/> -->
+  </transmission>
+  <transmission type="ardent_model/SimpleTransmission" name="t_tibia_${suffix}">
+    <joint name="t_tibia_${suffix}">
+    <actuator name="t_tibia_${suffix}">
+    <mechanicalReduction>1</mechanicalReduction>
+    <!-- <compensator k_belt="4000.0" mass_motor="0.05" kd_motor="15.0" lambda_motor="40.0" lambda_joint="40.0" lambda_combined="0.0"/> -->
+  </transmission>
+   <!-- <transmission name="t_coxa_${suffix}">
     <type>transmission_interface/SimpleTransmission</type>
     <joint name="j_coxa_${suffix}">
@@ -271,5 +289,5 @@
       <mechanicalReduction>1</mechanicalReduction>
     </actuator>
-  </transmission>
+  </transmission> -->
   <gazebo reference="MP_BODY">
     <material>Gazebo/Orange</material>

Commit message: Updated transmission interface handler

File: robot/urdf/ardent_urdf.xacro (robot description, xacro)
@@ -243,18 +243,18 @@
   </joint> -->
   <transmission type="ardent_model/SimpleTransmission" name="t_coxa_${suffix}">
-    <joint name="t_coxa_${suffix}">
-    <actuator name="t_coxa_${suffix}">
+    <joint name="j_coxa_${suffix}"/>
+    <actuator name="j_coxa_${suffix}_motor"/>
     <mechanicalReduction>1</mechanicalReduction>
     <!-- <compensator k_belt="4000.0" mass_motor="0.05" kd_motor="15.0" lambda_motor="40.0" lambda_joint="40.0" lambda_combined="0.0"/> -->
   </transmission>
   <transmission type="ardent_model/SimpleTransmission" name="t_femur_${suffix}">
-    <joint name="t_femur_${suffix}">
-    <actuator name="t_femur_${suffix}">
+    <joint name="j_femur_${suffix}"/>
+    <actuator name="j_femur_${suffix}_motor"/>
     <mechanicalReduction>1</mechanicalReduction>
     <!-- <compensator k_belt="4000.0" mass_motor="0.05" kd_motor="15.0" lambda_motor="40.0" lambda_joint="40.0" lambda_combined="0.0"/> -->
   </transmission>
   <transmission type="ardent_model/SimpleTransmission" name="t_tibia_${suffix}">
-    <joint name="t_tibia_${suffix}">
-    <actuator name="t_tibia_${suffix}">
+    <joint name="j_tibia_${suffix}"/>
+    <actuator name="j_tibia_${suffix}_motor"/>
     <mechanicalReduction>1</mechanicalReduction>
     <!-- <compensator k_belt="4000.0" mass_motor="0.05" kd_motor="15.0" lambda_motor="40.0" lambda_joint="40.0" lambda_combined="0.0"/> -->

Commit message: Controller Manager Integration

File: robot/urdf/ardent_urdf.xacro (robot description, xacro)
@@ -242,20 +242,35 @@
     <limit effort="2.8" velocity="5.6548668" lower="-2.6179939" upper="2.6179939" />
   </joint> -->
-  <transmission type="ardent_model/SimpleTransmission" name="t_coxa_${suffix}">
-    <joint name="j_coxa_${suffix}"/>
-    <actuator name="j_coxa_${suffix}_motor"/>
-    <mechanicalReduction>1</mechanicalReduction>
+  <transmission name="t_coxa_${suffix}">
+    <type>ardent/SimpleTransmission</type>
+    <joint name="j_coxa_${suffix}">
+      <hardwareInterface>hardware_interface/EffortJointInterface</hardwareInterface>
+    </joint>
+    <actuator name="j_coxa_${suffix}_motor">
+      <hardwareInterface>hardware_interface/EffortJointInterface</hardwareInterface>
+      <mechanicalReduction>1</mechanicalReduction>
+    </actuator>
     <!-- <compensator k_belt="4000.0" mass_motor="0.05" kd_motor="15.0" lambda_motor="40.0" lambda_joint="40.0" lambda_combined="0.0"/> -->
   </transmission>
-  <transmission type="ardent_model/SimpleTransmission" name="t_femur_${suffix}">
-    <joint name="j_femur_${suffix}"/>
-    <actuator name="j_femur_${suffix}_motor"/>
-    <mechanicalReduction>1</mechanicalReduction>
+  <transmission name="t_femur_${suffix}">
+    <type>ardent/SimpleTransmission</type>
+    <joint name="j_femur_${suffix}">
+      <hardwareInterface>hardware_interface/EffortJointInterface</hardwareInterface>
+    </joint>
+    <actuator name="j_femur_${suffix}_motor">
+      <hardwareInterface>hardware_interface/EffortJointInterface</hardwareInterface>
+      <mechanicalReduction>1</mechanicalReduction>
+    </actuator>
     <!-- <compensator k_belt="4000.0" mass_motor="0.05" kd_motor="15.0" lambda_motor="40.0" lambda_joint="40.0" lambda_combined="0.0"/> -->
   </transmission>
-  <transmission type="ardent_model/SimpleTransmission" name="t_tibia_${suffix}">
-    <joint name="j_tibia_${suffix}"/>
-    <actuator name="j_tibia_${suffix}_motor"/>
-    <mechanicalReduction>1</mechanicalReduction>
+  <transmission name="t_tibia_${suffix}">
+    <type>ardent/SimpleTransmission</type>
+    <joint name="j_tibia_${suffix}">
+      <hardwareInterface>hardware_interface/EffortJointInterface</hardwareInterface>
+    </joint>
+    <actuator name="j_tibia_${suffix}_motor">
+      <hardwareInterface>hardware_interface/EffortJointInterface</hardwareInterface>
+      <mechanicalReduction>1</mechanicalReduction>
+    </actuator>
     <!-- <compensator k_belt="4000.0" mass_motor="0.05" kd_motor="15.0" lambda_motor="40.0" lambda_joint="40.0" lambda_combined="0.0"/> -->
   </transmission>
